File: FT232RQ/FT232RQ.kicad_pcb (KiCad board)
At the start: 2 copper layers, 24 x 17 mm, 13 parts, among them IC1 FT232RQ, IC2 TLV74033PDBVR, J2 Conn_01x06_Male, P1 USB_C_Plug_USB2.0

Commit message: update PCB
tracks has been rerouted to make sure nobody cuts when manipulating the solder joint.
Routing:
- net GND: track 88.7 -> 70.0 mm
