File: CH340C/CH340C.kicad_pcb (KiCad board)
At the start: 2 copper layers, 24 x 17 mm, 19 parts, among them IC2 TLV74033PDBVR, J2 Conn_01x06_Male, P1 USB_C_Plug_USB2.0, U1 CH340C

Commit message: Update to v0.4
Parts:
- added JP2: SolderJumper_3_Bridged12, Jumper:SolderJumper-3_P1.3mm_Bridged12_RoundedPad1.0x1.5mm, B.Cu at (175.9, 73.6)
- moved G*** 2.52 mm to (181.9, 73.2)
- moved ? 0.20 mm to (167.6, 71.2)
Connections:
- J2 pad 4: +3V3 -> VCC
- U1 pad 16: +3V3 -> VCC
Routing:
- net +3V3: track 61.1 -> 23.5 mm, vias 5 -> 3
- net VCC: track 0.00 -> 18.8 mm, vias 0 -> 1
- net +5V: track 34.9 -> 43.5 mm, vias 2 -> 3
Other:
- board text added: "3.3/5v logic compatible"
- board text added: "5v"
- board text added: "FEB 2021 - v0.4"
- board text removed: "3.3v logic compatible"
- board text removed: "FEB 2021 - v0.3"

Commit message: update to v0.5
Parts:
- removed P1: USB_C_Plug_USB2.0, Connector_USB:USB_C_Receptacle_HRO_TYPE-C-31-M-12
- added J1: USB_C_Receptacle_USB2.0, Connector_USB:USB_C_Receptacle_HRO_TYPE-C-31-M-12, F.Cu at (183.2, 73.4)
Routing:
- net +5V: track 43.5 -> 23.3 mm, vias 3 -> 1
- net GND: track 52.6 -> 46.3 mm, vias 6 -> 0
- net D+: track 3.35 -> 7.76 mm, vias 0 -> 2
- net D-: track 2.85 -> 5.87 mm, vias 0 -> 2
- net +3V3: track 23.5 -> 26.5 mm, vias 3 -> 2
Other:
- board text added: "FEB 2021 - v0.5"
- board text removed: "FEB 2021 - v0.4"
