File: CH340C/CH340C.sch (KiCad schematic (older format))
At the start: 10 parts, among them IC2 TLV74033PDBVR, J2 Conn_01x06_Male, P1 USB_C_Plug_USB2.0, U1 CH340C

Commit message: Update to v0.4
Parts:
- added JP2: SolderJumper_3_Bridged12, Jumper:SolderJumper-3_P1.3mm_Bridged12_RoundedPad1.0x1.5mm, symbol Jumper:SolderJumper_3_Bridged12
Connections:
- net +3V3: now also JP2.1 (A); no longer J2.4 (Pin_4), U1.16 (VCC)
- net +5V: now also JP2.3 (B)
- new net VCC: J2.4 (Pin_4), JP2.2 (C), U1.16 (VCC)
Other:
- moved on the sheet: C5, C6, C7
Changed lines of the file:
@@
 Sheet 1 1
 Title "Candy UART"
-Date "2021-01-28"
-Rev "v0.2"
+Date "2021-02-04"
+Rev "v0.4"
 Comp "Upside Down Labs"
 Comment1 ""
 Comment2 "Candy size UART bridge"
-Comment3 "FT232RQ USB to UART Bridge"
-Comment4 "Candy UART - FTDI FT232RQ"
+Comment3 "CH340C USB to UART Bridge"
+Comment4 "Candy UART - CH340C"
 $EndDescr
 $Comp
@@
 Text Notes 9940 6430 2    157  ~ 31
 Pin Headers
-$Comp
-L power:+3V3 #PWR0122
-U 1 1 5FCB8801
-P 3240 4760
-F 0 "#PWR0122" H 3240 4610 50  0001 C CNN
-F 1 "+3V3" V 3240 5010 50  0000 C CNN
-F 2 "" H 3240 4760 50  0001 C CNN
-F 3 "" H 3240 4760 50  0001 C CNN
-	1    3240 4760
-	1    0    0    -1
-$EndComp
 Text GLabel 3640 5260 2    50   Input ~ 0
 CTS
@@
 L power:+5V #PWR0124
 U 1 1 6023D080
-P 8475 1080
-F 0 "#PWR0124" H 8475 930 50  0001 C CNN
-F 1 "+5V" H 8375 1230 50  0000 L CNN
-F 2 "" H 8475 1080 50  0001 C CNN
-F 3 "" H 8475 1080 50  0001 C CNN
-	1    8475 1080
+P 7765 1125
+F 0 "#PWR0124" H 7765 975 50  0001 C CNN
+F 1 "+5V" H 7665 1275 50  0000 L CNN
+F 2 "" H 7765 1125 50  0001 C CNN
+F 3 "" H 7765 1125 50  0001 C CNN
+	1    7765 1125
 	1    0    0    -1
 $EndComp
@@
 L power:GND #PWR0125
 U 1 1 6023DC28
-P 8475 1380
-F 0 "#PWR0125" H 8475 1130 50  0001 C CNN
-F 1 "GND" H 8480 1207 50  0000 C CNN
-F 2 "" H 8475 1380 50  0001 C CNN
-F 3 "" H 8475 1380 50  0001 C CNN
-	1    8475 1380
+P 7765 1425
+F 0 "#PWR0125" H 7765 1175 50  0001 C CNN
+F 1 "GND" H 7770 1252 50  0000 C CNN
+F 2 "" H 7765 1425 50  0001 C CNN
+F 3 "" H 7765 1425 50  0001 C CNN
+	1    7765 1425
 	1    0    0    -1
 $EndComp
@@
 L Device:C C6
 U 1 1 601D2719
-P 9150 1210
-F 0 "C6" H 9265 1256 50  0000 L CNN
-F 1 "100n" H 9265 1165 50  0000 L CNN
-F 2 "Capacitor_SMD:C_0805_2012Metric_Pad1.18x1.45mm_HandSolder" H 9188 1060 50  0001 C CNN
-F 3 "~" H 9150 1210 50  0001 C CNN
-	1    9150 1210
+P 8440 1255
+F 0 "C6" H 8555 1301 50  0000 L CNN
+F 1 "100n" H 8555 1210 50  0000 L CNN
+F 2 "Capacitor_SMD:C_0805_2012Metric_Pad1.18x1.45mm_HandSolder" H 8478 1105 50  0001 C CNN
+F 3 "~" H 8440 1255 50  0001 C CNN
+	1    8440 1255
 	1    0    0    -1
 $EndComp
@@
 L power:+3V3 #PWR0102
 U 1 1 601D443E
-P 9720 1050
-F 0 "#PWR0102" H 9720 900 50  0001 C CNN
-F 1 "+3V3" V 9720 1300 50  0000 C CNN
-F 2 "" H 9720 1050 50  0001 C CNN
-F 3 "" H 9720 1050 50  0001 C CNN
-	1    9720 1050
+P 9010 1095
+F 0 "#PWR0102" H 9010 945 50  0001 C CNN
+F 1 "+3V3" V 9010 1345 50  0000 C CNN
+F 2 "" H 9010 1095 50  0001 C CNN
+F 3 "" H 9010 1095 50  0001 C CNN
+	1    9010 1095
 	1    0    0    -1
 $EndComp
 Text GLabel 3140 4760 1    50   Input ~ 0
 V3
-Text GLabel 9150 1060 1    50   Input ~ 0
+Text GLabel 8440 1105 1    50   Input ~ 0
 V3
 $Comp
 L power:GND #PWR0103
 U 1 1 601D58A5
-P 9150 1360
-F 0 "#PWR0103" H 9150 1110 50  0001 C CNN
-F 1 "GND" V 9155 1232 50  0000 R CNN
-F 2 "" H 9150 1360 50  0001 C CNN
-F 3 "" H 9150 1360 50  0001 C CNN
-	1    9150 1360
+P 8440 1405
+F 0 "#PWR0103" H 8440 1155 50  0001 C CNN
+F 1 "GND" V 8445 1277 50  0000 R CNN
+F 2 "" H 8440 1405 50  0001 C CNN
+F 3 "" H 8440 1405 50  0001 C CNN
+	1    8440 1405
 	1    0    0    -1
 $EndComp
@@
 L power:GND #PWR0105
 U 1 1 601D66AD
-P 9720 1350
-F 0 "#PWR0105" H 9720 1100 50  0001 C CNN
-F 1 "GND" V 9725 1222 50  0000 R CNN
-F 2 "" H 9720 1350 50  0001 C CNN
-F 3 "" H 9720 1350 50  0001 C CNN
-	1    9720 1350
+P 9010 1395
+F 0 "#PWR0105" H 9010 1145 50  0001 C CNN
+F 1 "GND" V 9015 1267 50  0000 R CNN
+F 2 "" H 9010 1395 50  0001 C CNN
+F 3 "" H 9010 1395 50  0001 C CNN
+	1    9010 1395
 	1    0    0    -1
 $EndComp
@@
 L Device:C C5
 U 1 1 6023CB57
-P 8475 1230
-F 0 "C5" H 8590 1276 50  0000 L CNN
-F 1 "10u" H 8590 1185 50  0000 L CNN
-F 2 "Capacitor_SMD:C_0805_2012Metric_Pad1.18x1.45mm_HandSolder" H 8513 1080 50  0001 C CNN
-F 3 "~" H 8475 1230 50  0001 C CNN
-	1    8475 1230
+P 7765 1275
+F 0 "C5" H 7880 1321 50  0000 L CNN
+F 1 "10u" H 7880 1230 50  0000 L CNN
+F 2 "Capacitor_SMD:C_0805_2012Metric_Pad1.18x1.45mm_HandSolder" H 7803 1125 50  0001 C CNN
+F 3 "~" H 7765 1275 50  0001 C CNN
+	1    7765 1275
 	1    0    0    -1
 $EndComp
@@
 L Device:C C7
 U 1 1 601D40D9
-P 9720 1200
-F 0 "C7" H 9835 1246 50  0000 L CNN
-F 1 "10u" H 9835 1155 50  0000 L CNN
-F 2 "Capacitor_SMD:C_0805_2012Metric_Pad1.18x1.45mm_HandSolder" H 9758 1050 50  0001 C CNN
-F 3 "~" H 9720 1200 50  0001 C CNN
-	1    9720 1200
+P 9010 1245
+F 0 "C7" H 9125 1291 50  0000 L CNN
+F 1 "10u" H 9125 1200 50  0000 L CNN
+F 2 "Capacitor_SMD:C_0805_2012Metric_Pad1.18x1.45mm_HandSolder" H 9048 1095 50  0001 C CNN
+F 3 "~" H 9010 1245 50  0001 C CNN
+	1    9010 1245
 	1    0    0    -1
 $EndComp
@@
 TXD
 $Comp
-L power:+3V3 #PWR0108
-U 1 1 601CC292
-P 9320 5075
-F 0 "#PWR0108" H 9320 4925 50  0001 C CNN
-F 1 "+3V3" V 9320 5325 50  0000 C CNN
-F 2 "" H 9320 5075 50  0001 C CNN
-F 3 "" H 9320 5075 50  0001 C CNN
-	1    9320 5075
-	0    -1   -1   0
-$EndComp
-$Comp
 L Connector:Conn_01x06_Male J2
 U 1 1 5FC71350
@@
 Text GLabel 8820 4775 1    50   Input ~ 0
 CTS
+$Comp
+L Jumper:SolderJumper_3_Bridged12 JP2
+U 1 1 601C0192
+P 10560 1155
+F 0 "JP2" V 10606 1223 50  0000 L CNN
+F 1 "SolderJumper_3_Bridged12" V 10515 1223 50  0000 L CNN
+F 2 "Jumper:SolderJumper-3_P1.3mm_Bridged12_RoundedPad1.0x1.5mm" H 10560 1155 50  0001 C CNN
+F 3 "~" H 10560 1155 50  0001 C CNN
+	1    10560 1155
+	0    -1   -1   0
+$EndComp
+$Comp
+L power:+3V3 #PWR0108
+U 1 1 601CB740
+P 10560 1355
+F 0 "#PWR0108" H 10560 1205 50  0001 C CNN
+F 1 "+3V3" V 10560 1575 50  0000 C CNN
+F 2 "" H 10560 1355 50  0001 C CNN
+F 3 "" H 10560 1355 50  0001 C CNN
+	1    10560 1355
+	-1   0    0    1
+$EndComp
+Text GLabel 10710 1155 2    50   Input ~ 0
+VCC
+$Comp
+L power:+5V #PWR0113
+U 1 1 601D2B87
+P 10560 955
+F 0 "#PWR0113" H 10560 805 50  0001 C CNN
+F 1 "+5V" H 10460 1105 50  0000 L CNN
+F 2 "" H 10560 955 50  0001 C CNN
+F 3 "" H 10560 955 50  0001 C CNN
+	1    10560 955
+	1    0    0    -1
+$EndComp
+Text GLabel 9320 5075 0    50   Input ~ 0
+VCC
+Text GLabel 3240 4760 1    50   Input ~ 0
+VCC
 $EndSCHEMATC

Commit message: update to v0.5
Parts:
- removed P1: USB_C_Plug_USB2.0, Connector_USB:USB_C_Receptacle_HRO_TYPE-C-31-M-12, symbol Connector:USB_C_Plug_USB2.0
- added J1: USB_C_Receptacle_USB2.0, Connector_USB:USB_C_Receptacle_HRO_TYPE-C-31-M-12, symbol Connector:USB_C_Receptacle_USB2.0
Connections:
- net +5V: now also J1.A4 (VBUS), J1.A9 (VBUS), J1.B4 (VBUS), J1.B9 (VBUS)
- net D+: now also J1.A6 (D+), J1.B6 (D+)
- net D-: now also J1.A7 (D-), J1.B7 (D-)
- net GND: now also J1.A1 (GND), J1.A12 (GND), J1.B1 (GND), J1.B12 (GND), J1.S1 (SHIELD)
Changed lines of the file:
@@
 Sheet 1 1
 Title "Candy UART"
-Date "2021-02-04"
-Rev "v0.4"
+Date "2021-02-18"
+Rev "v0.5"
 Comp "Upside Down Labs"
 Comment1 ""
@@
 $EndDescr
 $Comp
-L Connector:USB_C_Plug_USB2.0 P1
-U 1 1 5FC51652
-P 3600 1830
-F 0 "P1" H 3600 2730 50  0000 C CNN
-F 1 "USB_C_Plug_USB2.0" H 3600 2630 50  0000 C CNN
-F 2 "Connector_USB:USB_C_Receptacle_HRO_TYPE-C-31-M-12" H 3750 1830 50  0001 C CNN
-F 3 "https://www.usb.org/sites/default/files/documents/usb_type-c.zip" H 3750 1830 50  0001 C CNN
-	1    3600 1830
-	1    0    0    -1
-$EndComp
-$Comp
 L power:GND #PWR0101
 U 1 1 5FC58946
-P 3600 2730
-F 0 "#PWR0101" H 3600 2480 50  0001 C CNN
-F 1 "GND" H 3605 2557 50  0000 C CNN
-F 2 "" H 3600 2730 50  0001 C CNN
-F 3 "" H 3600 2730 50  0001 C CNN
-	1    3600 2730
-	1    0    0    -1
-$EndComp
-Text GLabel 4200 1730 2    50   Input ~ 0
+P 3700 2570
+F 0 "#PWR0101" H 3700 2320 50  0001 C CNN
+F 1 "GND" H 3705 2397 50  0000 C CNN
+F 2 "" H 3700 2570 50  0001 C CNN
+F 3 "" H 3700 2570 50  0001 C CNN
+	1    3700 2570
+	1    0    0    -1
+$EndComp
+Text GLabel 4300 1670 2    50   Input ~ 0
 D-
-Text GLabel 4200 1930 2    50   Input ~ 0
+Text GLabel 4300 1770 2    50   Input ~ 0
 D+
 Text GLabel 2840 5360 0    50   Input ~ 0
@@
 L power:+5V #PWR0109
 U 1 1 5FCA1CB3
-P 4200 1230
-F 0 "#PWR0109" H 4200 1080 50  0001 C CNN
-F 1 "+5V" V 4215 1358 50  0000 L CNN
-F 2 "" H 4200 1230 50  0001 C CNN
-F 3 "" H 4200 1230 50  0001 C CNN
-	1    4200 1230
+P 4300 1070
+F 0 "#PWR0109" H 4300 920 50  0001 C CNN
+F 1 "+5V" V 4315 1198 50  0000 L CNN
+F 2 "" H 4300 1070 50  0001 C CNN
+F 3 "" H 4300 1070 50  0001 C CNN
+	1    4300 1070
 	0    1    1    0
 $EndComp
@@
 L power:GND #PWR0121
 U 1 1 602306E2
-P 3300 2730
-F 0 "#PWR0121" H 3300 2480 50  0001 C CNN
-F 1 "GND" H 3305 2557 50  0000 C CNN
-F 2 "" H 3300 2730 50  0001 C CNN
-F 3 "" H 3300 2730 50  0001 C CNN
-	1    3300 2730
+P 3400 2570
+F 0 "#PWR0121" H 3400 2320 50  0001 C CNN
+F 1 "GND" H 3405 2397 50  0000 C CNN
+F 2 "" H 3400 2570 50  0001 C CNN
+F 3 "" H 3400 2570 50  0001 C CNN
+	1    3400 2570
 	1    0    0    -1
 $EndComp
@@
 	1    0    0    -1
 $EndComp
-NoConn ~ 4200 1430
-NoConn ~ 4200 1530
+NoConn ~ 4300 1370
+NoConn ~ 4300 1270
 NoConn ~ 3640 5360
 NoConn ~ 3640 5460
@@
 Text GLabel 3240 4760 1    50   Input ~ 0
 VCC
+$Comp
+L Connector:USB_C_Receptacle_USB2.0 J1
+U 1 1 602E3FEE
+P 3700 1670
+F 0 "J1" H 3807 2537 50  0000 C CNN
+F 1 "USB_C_Receptacle_USB2.0" H 3807 2446 50  0000 C CNN
+F 2 "Connector_USB:USB_C_Receptacle_HRO_TYPE-C-31-M-12" H 3850 1670 50  0001 C CNN
+F 3 "https://www.usb.org/sites/default/files/documents/usb_type-c.zip" H 3850 1670 50  0001 C CNN
+	1    3700 1670
+	1    0    0    -1
+$EndComp
+Text GLabel 4300 1570 2    50   Input ~ 0
+D-
+Text GLabel 4300 1870 2    50   Input ~ 0
+D+
 $EndSCHEMATC
